File: kicad/UFI_Modular.kicad_pcb (KiCad board)
At the start: 4 copper layers, 110.1 x 85 mm, 38 parts, among them J1 FDD1, J10 GbE, J12 NVMe, J13 EXP40, J14 MOD, J15 MOD_USB, J16 12V, J17 SWD, J2 FDD2, J3 Apple, J4 Amiga, J5 IEC, J6 CM5_A, J7 CM5_B, J8 PWR, J9 PC, SW1 RST, SW2 BOOT, U1 STM32H723, U10 TPS54331, U11 TPS54331, U2 W25Q128, U20 74LVC245, U21 74LVC245, U22 74LVC245, U23 74LVC245, Y1 25MHz, Y2 32.768k

Commit message: kicad: UFI_Modular layout changes, KiCad 10 re-save of the other boards
UFI_Modular.kicad_pcb/.kicad_pro carry layout work; the remaining
schematics, boards, footprints and UFI.kicad_pro are re-saves by
KiCad 10 (format/default-settings updates).
Other:
- board size 110.1 x 85 mm -> 110 x 85 mm
- net class Default removed
- net class Ethernet removed
- net class Power removed
- net class USB_HS removed
