File: kicad/UFI_Headless/UFI_Headless.kicad_sch (KiCad schematic)
At the start: 0 parts

Commit message: v0.7: Apple Disk II port (J14/J15), board 110 x 97 mm; firmware 1.11: drives apple/apple2
Board
- Apple_Port sheet: J14 2x10 (Disk II controller pinout), SN74AHCT244 outputs at FDD_5V
  (phases, /ENABLE 1+2, /WRREQ, WRDATA), 74LVC2G17 inputs (RDDATA, WRPROT), ICL7662 -12V
  from FDD_12V, reset-safe 10k arrays, ESD on all port lines, J15 = /ENABLE drive 2
- MCU: RDDATA PA2 (TIM2_CH3), WRDATA PA7 (TIM3_CH2), PH0/1/3 PF12/13/15, PH2 PG6,
  EN1 PG5, EN2 PB12, WRREQ PB14, WRPROT PB15; board ID 10k/2.2k = v0.7
- outline +12 mm (eco/extend_outline.py), mounting holes H5/H6, ECO + Freerouting, hand
  routes for EN1/PH2 (PB11/PF14 unreachable), FDD_12V to J14/U18, D16 GND via;
  J14 uses a project copy of the IDC footprint (silk edge clears the J7 pin-1 mark)
- DRC 0 incl. warnings, unconnected 0, parity 0, via-in-pad 0; fab outputs regenerated

Firmware 1.11
- Disk II stepper (4 phases, half tracks, recalibrate = 80 half steps to the stop, phases
  off between seeks), /ENABLE = motor, write protect, no disk change / always ready
- capture input switch CH1/CH3 (DMAMUX), Apple reads in 200 ms slices (no index)
- writes: TIM3_CH2 toggle mode, /WRREQ, start without index, no precomp; erase = /WRREQ
- Apple drives selectable only on a v0.7 board (board ID); UFI.CFG drive=apple/apple2,
  SCP disk type Apple II without index flag; host drive name apple2
- dump simulation: SCP still byte-identical; host tests pass

Docs: README Apple section + GPIO table, bring-up 7.2f-7.2j, order list v0.7
Other:
- added sheet Apple_Port (Apple_Port.kicad_sch)
- note added: "UFI Headless - STM32H723 flux engine without CM5. Sheets: Power, MCU_Core, Flux_Interface, FDD_Connectors, IEC_Bus, Apple_Port."
- note removed: "UFI Headless - STM32H723 flux engine without CM5. Sheets: Power, MCU_Core, Flux_Interface, FDD_Connectors, IEC_Bus."
Changed lines of the file:
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@@
 (paper "A3")
 (title_block (title "UFI Headless") (date "2026-10-05") (rev "0.1") (company "UFI Project"))
-(text "UFI Headless - STM32H723 flux engine without CM5.\nSheets: Power, MCU_Core, Flux_Interface, FDD_Connectors, IEC_Bus." (exclude_from_sim no) (at 20 20 0) (effects (font (size 2 2)) (justify left top)))
+(text "UFI Headless - STM32H723 flux engine without CM5.\nSheets: Power, MCU_Core, Flux_Interface, FDD_Connectors, IEC_Bus, Apple_Port." (exclude_from_sim no) (at 20 20 0) (effects (font (size 2 2)) (justify left top)))
 (sheet (at 30 50) (size 50 30) (fields_autoplaced yes) (stroke (width 0.1524) (type solid)) (fill (color 0 0 0 0.0000)) (property "Sheetname" "Power" (at 30 49.3 0) (effects (font (size 1.27 1.27)) (justify left bottom))) (property "Sheetfile" "Power.kicad_sch" (at 30 80.6 0) (effects (font (size 1.27 1.27)) (justify left top))) (instances (project "UFI_Headless" (path "/dc1b800d-cedf-5627-97f0-e6992ff33669" (page "2")))))
 (sheet (at 100 50) (size 50 30) (fields_autoplaced yes) (stroke (width 0.1524) (type solid)) (fill (color 0 0 0 0.0000)) (property "Sheetname" "MCU_Core" (at 100 49.3 0) (effects (font (size 1.27 1.27)) (justify left bottom))) (property "Sheetfile" "MCU_Core.kicad_sch" (at 100 80.6 0) (effects (font (size 1.27 1.27)) (justify left top))) (instances (project "UFI_Headless" (path "/dc1b800d-cedf-5627-97f0-e6992ff33669" (page "3")))))
@@
 (sheet (at 240 50) (size 50 30) (fields_autoplaced yes) (stroke (width 0.1524) (type solid)) (fill (color 0 0 0 0.0000)) (property "Sheetname" "FDD_Connectors" (at 240 49.3 0) (effects (font (size 1.27 1.27)) (justify left bottom))) (property "Sheetfile" "FDD_Connectors.kicad_sch" (at 240 80.6 0) (effects (font (size 1.27 1.27)) (justify left top))) (instances (project "UFI_Headless" (path "/dc1b800d-cedf-5627-97f0-e6992ff33669" (page "5")))))
 (sheet (at 310 50) (size 50 30) (fields_autoplaced yes) (stroke (width 0.1524) (type solid)) (fill (color 0 0 0 0.0000)) (property "Sheetname" "IEC_Bus" (at 310 49.3 0) (effects (font (size 1.27 1.27)) (justify left bottom))) (property "Sheetfile" "IEC_Bus.kicad_sch" (at 310 80.6 0) (effects (font (size 1.27 1.27)) (justify left top))) (instances (project "UFI_Headless" (path "/dc1b800d-cedf-5627-97f0-e6992ff33669" (page "6")))))
+(sheet (at 380 50) (size 50 30) (fields_autoplaced yes) (stroke (width 0.1524) (type solid)) (fill (color 0 0 0 0.0000)) (property "Sheetname" "Apple_Port" (at 380 49.3 0) (effects (font (size 1.27 1.27)) (justify left bottom))) (property "Sheetfile" "Apple_Port.kicad_sch" (at 380 80.6 0) (effects (font (size 1.27 1.27)) (justify left top))) (instances (project "UFI_Headless" (path "/dc1b800d-cedf-5627-97f0-e6992ff33669" (page "7")))))
 (sheet_instances (path "/" (page "1")))
 )
