File: kicad/UFI_Headless/Power.kicad_sch (KiCad schematic)
At the start: 68 parts, among them J1 USB-C, J16 USB_HDR, J17 PSU_IN, J2 12V DC 5.5/2.1, J3 FDD_PWR, Q1 AO3401A, Q2 2N7002, Q3 AO3401A, Q4 2N7002, U1 USBLC6-2SC6, U12 INA180A1, U13 INA180A1, U19 TPS2116DRL, U2 TPS54202DDC, U3 TPS2116DRL, U4 AP7361C-33E

Commit message: KiCad v0.7 rework, stage A9a (owner review of 2026-10-24, protection items before the B3 re-layout): J17 PSU-IN and J3 drive power become keyed JST XH B4B-XH-A (LCSC C144395, 3 A, same pin order 1 +5V 2/3 GND 4 +12V) because a reversed 2.54-mm header would have put 12 V on U19 (6 V max) or on the drive's 5 V input - adapter cables Berg <-> XH described in kicad/UFI_Headless/docs/Inbetriebnahme.md; D27 SS54 (C16103) from J17 pin 4 (new local net +12V_PSU) to +12V as a diode-OR with D2, so the jack and the C64 PSU may be plugged at once; U24 USBLC6-2SC6 (C7519, VRWM 5.25 V) on CC1/CC2 next to J1 (the USBLC6 U1 only covers D+/D-); R125-R127 220 R (C22962) in series on the GUARD cable, cable side GUARD_OFF_J/GUARD_ERR5_J/GUARD_ERR12_J, MCU side unchanged with the 10k pull-ups; R26/R29 0.1 R -> 50 mR 1 % (TA-I RLM12FTCMR050 C912768, alternative Panasonic ERJ8CWFR050V C713437, stock to be checked in stage C) and F2 1206 -> 1812 like F3 (C20999) to cut the series resistance of the 5 V drive chain; SW3/SW4 (DNP buttons A/B) deleted from the schematic incl. their labels and GND symbols, buttons stay on the front header J12 pin 13/14. Firmware in the same commit: ufi_board.c scales the INA180 reading by board revision (v1.0 50 mR = 1 mV/mA, v0.x 0.1 R = 2 mV/mA via ufi_board_rev()), comments in board.h; protocol doc BOARD_STATUS mA fields note the scale. ERC over the whole project 0 errors / 0 warnings (build/erc.rpt refreshed, it had been from 7.10. without the LAN sheet); ARM build 0 warnings, AXI free 36688 B unchanged; offline gate: all 23 check groups green, the final pytest step of the owner's check_all.py reports "No module named pytest" in this environment (not related to this change). fertigung/: the v0.x Gerber/BOM/CPL/zip of 7.10. removed (README stub explains), nothing may be ordered before stage C. PLAN.md: row A9 with the owner's ten-point definition (A9a done; A9b write-protect default-on + INDEX on TIM2_CH4 + pin map, A9c soft start + RTC open), B3 row; kicad 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
Parts:
- added D27: SS54, Diode_SMD:D_SMC, symbol Device:D_Schottky
- added U24: USBLC6-2SC6, Package_TO_SOT_SMD:SOT-23-6, symbol Power_Protection:USBLC6-2SC6
- F2: value 1.1A hold 6V -> 1.1A hold 24V; footprint Fuse:Fuse_1206_3216Metric -> Fuse:Fuse_1812_4532Metric; LCSC C20801 -> C20999; MPN SMD1206P110TF (1.1A hold, 6V) -> SMD1812P110TF/24 (1.1A hold, 24V, same part as F3; 1812 has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
- J17: footprint Connector_PinHeader_2.54mm:PinHeader_1x04_P2.54mm_Vertical -> Connector_JST:JST_XH_B4B-XH-A_1x04_P2.50mm_Vertical; LCSC C32713270 -> C144395; MPN (none) -> JST B4B-XH-A(LF)(SN) (XH 2.5 mm, 3 A, keyed); Note PC PSU floppy (Berg) plug: 1 +5V, 2/3 GND, 4 +12V -> C64 PSU in, keyed XH housing on the cable: 1 +5V, 2/3 GND, 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
- J3: footprint Connector_PinHeader_2.54mm:PinHeader_1x04_P2.54mm_Vertical -> Connector_JST:JST_XH_B4B-XH-A_1x04_P2.50mm_Vertical; LCSC C32713270 -> C144395; MPN (none) -> JST B4B-XH-A(LF)(SN) (XH 2.5 mm, 3 A, keyed); Note Pin1 +5V, 2/3 GND, 4 +12V (Berg/Molex FDD order) -> drive power out, keyed XH housing on the cable to the drive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
- R26, R29: value 0.1R 1% -> 0.05R 1%; LCSC C25334 -> C912768; MPN 1206W4F100LT5E (0.1R 1% 1/4W) -> RLM12FTCMR050 (50 mR 1% 1 W, TA-I; alternative Panasonic ER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; Note (none) -> INA180A1 (20 V/V): 1 V per A, 1.5 V at 1.5 A; Kelvin connec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
Connections:
- net +12V: now also D27.1 (K)
- net +12V_IN: no longer J17.4 (Pin_4)
- net CC1: now also U24.1 (I/O1), U24.6 (I/O1)
- net CC2: now also U24.3 (I/O2), U24.4 (I/O2)
- net GND: now also U24.2 (GND)
- net VBUS: now also U24.5 (VBUS)
- new net +12V_PSU: D27.2 (A), J17.4 (Pin_4)
