File: kicad/UFI_Headless/LAN.kicad_sch (KiCad schematic)
At the start: 35 parts, among them J22 HR911105A, U23 W5500, Y2 25MHz CL=12pF

Commit message: KiCad v0.7 rework, stage C part 1 (BOM completion before the release, review note H12): every BOM row now carries an LCSC number, checked against the JLCPCB SMT catalogue on 2026-10-25 (stock in brackets). LAN sheet: U23 W5500 C32843 (9019), J22 HR911105A C12074 (72229, THT), Y2 25 MHz 12 pF +-10 ppm YXC X322525MOB4SI C9006 (basic; load capacitance 12 pF verified on the LCSC parameter page, fits the 18 pF C59/C60), C59/C60 18 pF C0G Yageo CC0603JRNPO9BN180 C107040, C61/C74 10 nF FH 0603B103K500NT C57112 (basic), C71 22 nF Samsung CL10B223KB8NNNC C21122 (basic), C72/C73 6.8 nF FH 0603B682K500NT C1631 (basic), C62 4.7 uF C1779, C63/C69 10 uF C15850, C64-C68/C70 100 nF C14663, FB2 C1002, R109 1M C22935, R111 12.4k 1 % C22865, R112/R113 49.9R 1 % C23185 (basic), R114 10R 1 % C22859 (basic), R115/R116 82R 1 % C23255, R117/R118 330R C23138, R119-R124 10k C25804. Other sheets: R75-R99/R105/R128 1k C21190, R74/R107/R108 10k C25804, R101-R104/R130 470R C23179, R106/R131 100k C25803, C58 100 nF C14663 (value text 100n -> 100nF so it groups with the other 100 nF), D18-D26/D28/D29 PESD3V3L1BA C51450 (48710) like D32-D34, Q5 2N7002 C8545 (basic), U22 TS5A3166DBVR C353035 (10678), J2 DC-005 2.0 C16214 (92305; same pin pattern as the KiCad BarrelJack_Horizontal footprint, placement to be checked in the JLC viewer), J7 2x12 IDC ZHOURI DC3-2.54-24PAS C5144580 (stock 81 - hand soldering stays the recommendation in docs/Bestellung_JLC.md), J12 2x8 IDC DC3-2.54-16PAS C2977594 (4335), J16 2x5 pin header XFCN PZ254V-12-10P C492422 (105667), J21 2x10 pin header PZ254V-12-20P C492427 (63622). Solder jumpers JP5-JP8 are excluded from the BOM (in_bom no) like JP1/JP3 - bare copper, nothing to place. Stock of the review's watch list: U9 SN74LS07DR C371970 4776, D31 ESDA6V1-5SC6 C6650 3010, L1 SRN6045TA-150M C1330797 1866. BOM export (kicad-cli sch export bom, grouped by value/footprint/LCSC): 99 rows, 0 without LCSC, 0 DNP. ERC over the whole project 0 errors / 0 warnings (build/erc.rpt). No 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
Parts:
- C59, C60: LCSC (none) -> C107040
- C61, C74: LCSC (none) -> C57112
- C62: LCSC (none) -> C1779
- C63, C69: LCSC (none) -> C15850
- C64, C65, C66, C67, C68, C70: LCSC (none) -> C14663
- C71: LCSC (none) -> C21122
- C72, C73: LCSC (none) -> C1631
- FB2: LCSC (none) -> C1002
- J22: LCSC (none) -> C12074
- R109: LCSC (none) -> C22935
- R111: LCSC (none) -> C22865
- R112, R113: LCSC (none) -> C23185
- R114: LCSC (none) -> C22859
- R115, R116: LCSC (none) -> C23255
- R117, R118: LCSC (none) -> C23138
- R119, R120, R121, R122, R123, R124: LCSC (none) -> C25804
- U23: LCSC (none) -> C32843
- Y2: LCSC (none) -> C9006
