File: kicad/UFI_Headless/Flux_Interface.kicad_sch (KiCad schematic)
At the start: 55 parts, among them Q10 BSS138DW, Q11 BSS138DW, Q5 2N7002, Q6 BSS138DW, Q7 BSS138DW, Q8 BSS138DW, Q9 BSS138DW, U14 74LVC1G32, U22 TS5A3166DBVR, U30 74LVC2G32, U31 74LVC1G02, U8 74LVC14AD

Commit message: U31 74LVC1G02 (write-lock NOR, A11f): LCSC C52953351 (MDD) -> C113520 (TI SN74LVC1G02DCKR, SOT-353/SC-70-5, stock 38012 on 2026-10-26). JLC has no footprint/3D model for the MDD part yet and would only create it after payment (+1 day, no placement check possible beforehand). Same standard pinout (1 A, 2 B, 3 GND, 4 Y, 5 VCC), footprint unchanged, no net change. ERC 0/0 (fertigung/erc.rpt), JLC BOM and KiCad BOM regenerated. The A11f rows in README/PLAN keep the original part as history.
Claude-Session: https://claude.ai/code/session_014MdzrcyXuayppPHbfEjUrw
Parts:
- U31: LCSC C52953351 -> C113520
Changed lines of the file:
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@@
 			)
 		)
-    (property "LCSC" "C52953351" (at 119.38 378.46 0)
+    (property "LCSC" "C113520" (at 119.38 378.46 0)
       (effects (font (size 1.27 1.27)) (hide yes))
     )
